File: hardware/spot.kicad_pcb (KiCad board)
At the start: 6 copper layers, 50 x 50 mm, 50 parts, among them J1001 NE8FAV, J101 Cortex, J102 DX07S016JA3, J103 WAGO 2065-100, J104 WAGO 2065-100, J105 WAGO 2065-100, J901 NE8FAV, Q101 BSC010N04LS, Q102 BSC010N04LS, SW101 SKSG, U1001 THVD2442, U101 ATSAMD51J, U102 TPS78433QWDRBRQ1, U301 TPSM33620S5QRDNRQ1, U901 THVD2442, Y101 32k768

Commit message: Update LDO
Connections:
- U102 pad 6: unconnected-(U102-Pad6) -> +5V
