File: hardware/spot.kicad_pcb (KiCad board)
At the start: 6 copper layers, 50 x 50 mm, 50 parts, among them J1001 NE8FAV, J101 Cortex, J102 DX07S016JA3, J103 WAGO 2065-100, J104 WAGO 2065-100, J105 WAGO 2065-100, J901 NE8FAV, Q101 BSC010N04LS, Q102 BSC010N04LS, SW101 SKSG, U1001 THVD2442, U101 ATSAMD51J, U102 TPS78433QWDRBRQ1, U301 TPSM33620S5QRDNRQ1, U901 THVD2442, Y101 32k768

Commit message: Rename
Changed lines of the file:
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@@
 	(paper "A4")
 	(title_block
-		(date "2026-08-20")
+		(date "2026-08-30")
 		(rev "2026-08-20")
 	)
@@
 		)
 		(sheetname "/Link Socket/")
-		(sheetfile "LinkSocket.kicad_sch")
+		(sheetfile "Link-Socket.kicad_sch")
 		(attr smd)
 		(duplicate_pad_numbers_are_jumpers no)
@@
 		(property ki_fp_filters "C_*")
 		(sheetname "/Link Plug/")
-		(sheetfile "LinkPlug.kicad_sch")
+		(sheetfile "Link-Plug.kicad_sch")
 		(attr smd)
 		(duplicate_pad_numbers_are_jumpers no)
@@
 		(property ki_fp_filters "C_*")
 		(sheetname "/Power +5V/")
-		(sheetfile "PowerSupply.kicad_sch")
+		(sheetfile "Power-DCDC.kicad_sch")
 		(attr smd)
 		(duplicate_pad_numbers_are_jumpers no)
@@
 		(property ki_fp_filters "C_*")
 		(sheetname "/Power +5V/")
-		(sheetfile "PowerSupply.kicad_sch")
+		(sheetfile "Power-DCDC.kicad_sch")
 		(attr smd)
 		(duplicate_pad_numbers_are_jumpers no)
@@
 		)
 		(sheetname "/Power +5V/")
-		(sheetfile "PowerSupply.kicad_sch")
+		(sheetfile "Power-DCDC.kicad_sch")
 		(attr smd)
 		(duplicate_pad_numbers_are_jumpers no)
@@
 		(property ki_fp_filters "C_*")
 		(sheetname "/Link Socket/")
-		(sheetfile "LinkSocket.kicad_sch")
+		(sheetfile "Link-Socket.kicad_sch")
 		(attr smd)
 		(duplicate_pad_numbers_are_jumpers no)
@@
 		(property ki_fp_filters "C_*")
 		(sheetname "/Power +5V/")
-		(sheetfile "PowerSupply.kicad_sch")
+		(sheetfile "Power-DCDC.kicad_sch")
 		(attr smd)
 		(duplicate_pad_numbers_are_jumpers no)
@@
 		)
 		(sheetname "/Link Plug/")
-		(sheetfile "LinkPlug.kicad_sch")
+		(sheetfile "Link-Plug.kicad_sch")
 		(attr smd)
 		(duplicate_pad_numbers_are_jumpers no)
@@
 		(property ki_fp_filters "C_*")
 		(sheetname "/Power +5V/")
-		(sheetfile "PowerSupply.kicad_sch")
+		(sheetfile "Power-DCDC.kicad_sch")
 		(attr smd)
 		(duplicate_pad_numbers_are_jumpers no)
@@
 		(property ki_fp_filters "C_*")
 		(sheetname "/Power +5V/")
-		(sheetfile "PowerSupply.kicad_sch")
+		(sheetfile "Power-DCDC.kicad_sch")
 		(attr smd)
 		(duplicate_pad_numbers_are_jumpers no)
@@
 		(property ki_fp_filters "R_*")
 		(sheetname "/Link Socket/")
-		(sheetfile "LinkSocket.kicad_sch")
+		(sheetfile "Link-Socket.kicad_sch")
 		(attr smd)
 		(duplicate_pad_numbers_are_jumpers no)
@@
 		(property ki_fp_filters "R_*")
 		(sheetname "/Link Plug/")
-		(sheetfile "LinkPlug.kicad_sch")
+		(sheetfile "Link-Plug.kicad_sch")
 		(attr smd)
 		(duplicate_pad_numbers_are_jumpers no)
@@
 		)
 		(sheetname "/Link Socket/")
-		(sheetfile "LinkSocket.kicad_sch")
+		(sheetfile "Link-Socket.kicad_sch")
 		(attr through_hole allow_missing_courtyard)
 		(duplicate_pad_numbers_are_jumpers no)
@@
 		)
 		(sheetname "/Link Plug/")
-		(sheetfile "LinkPlug.kicad_sch")
+		(sheetfile "Link-Plug.kicad_sch")
 		(attr through_hole allow_missing_courtyard)
 		(duplicate_pad_numbers_are_jumpers no)
