File: hardware/spot.kicad_sch (KiCad schematic)
At the start: 36 parts, among them J101 Cortex, J102 DX07S016JA3, J103 WAGO 2065-100, J104 WAGO 2065-100, J105 WAGO 2065-100, Q101 BSC010N04LS, Q102 BSC010N04LS, SW101 SKSG, U101 ATSAMD51J, U102 TPS78433QWDRBRQ1, Y101 32k768

Commit message: Update LDO
Connections:
- net +5V: now also U102.6 (EN)
Changed lines of the file:
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@@
 	(title_block
 		(title "V2 spot")
-		(date "2026-06-30")
-		(rev "2026-06-30")
+		(date "2026-08-20")
+		(rev "2026-08-20")
 		(company "Versio Duo")
 		(comment 1 "LED Light")
@@
 		(unit 1)
 		(body_style 1)
-		(exclude_from_sim yes)
+		(exclude_from_sim no)
 		(in_bom no)
 		(on_board yes)
@@
 			(at 240.03 167.64 0)
 			(hide yes)
+			(show_name no)
+			(do_not_autoplace no)
+			(effects
+				(font
+					(size 1.27 1.27)
+				)
+			)
+		)
+		(property "Sim.Enable" "0"
+			(at 240.03 167.64 0)
+			(hide yes)
