File: hardware/spot.kicad_sch (KiCad schematic)
At the start: 36 parts, among them J101 Cortex, J102 DX07S016JA3, J103 WAGO 2065-100, J104 WAGO 2065-100, J105 WAGO 2065-100, Q101 BSC010N04LS, Q102 BSC010N04LS, SW101 SKSG, U101 ATSAMD51J, U102 TPS78433QWDRBRQ1, Y101 32k768

Commit message: Rename
Other:
- sheet Link Plug: file LinkPlug.kicad_sch -> Link-Plug.kicad_sch
- sheet Link Socket: file LinkSocket.kicad_sch -> Link-Socket.kicad_sch
- sheet Power +5V: file PowerSupply.kicad_sch -> Power-DCDC.kicad_sch
