File: hardware/Link-Plug.kicad_sch (KiCad schematic)
At the start: 4 parts, among them J1001 NE8FAV, U1001 THVD2442

Commit message: Rename
Parts:
- removed C1001: 0u1, V2_Capacitor_SMD:C_1608, symbol V2_Capacitor:1608_0u1
- removed J1001: NE8FAV, V2_Connector_EtherCon:NE8FAV, symbol V2_Connector_EtherCon:NE8FAV
- removed R1001: 100R, V2_Resistor_SMD:R_1608, symbol V2_Resistor:1608_100R
- removed U1001: THVD2442, V2_Package_SON:VSON-10-4-1EP_3x3mm_P0.5mm_EP1.65x2.4mm_ThermalVias, symbol V2_Interface_RS485:THVD2442
- added C901: 0u1, V2_Capacitor_SMD:C_1608, symbol V2_Capacitor:1608_0u1
- added J901: NE8FAV, V2_Connector_EtherCon:NE8FAV, symbol V2_Connector_EtherCon:NE8FAV
- added R901: 100R, V2_Resistor_SMD:R_1608, symbol V2_Resistor:1608_100R
- added U901: THVD2442, V2_Package_SON:VSON-10-4-1EP_3x3mm_P0.5mm_EP1.65x2.4mm_ThermalVias, symbol V2_Interface_RS485:THVD2442
Connections:
- net +3V3: now also C901.1, U901.10 (VCC)
- net GND: now also C901.2, J901.7, J901.8, U901.11 (GND), U901.5 (GND)
- net Power: now also J901.4, J901.5
- net RX: now also U901.1 (R)
- net RX-A: now also J901.3, R901.1, U901.9 (A)
- net RX-B: now also J901.6, R901.2, U901.8 (B)
- net RX-Enable: now also U901.2 (RE)
- net Shield: now also J901.S
- net TX: now also U901.4 (D)
- net TX-Enable: now also U901.3 (DE)
- net TX-Y: now also J901.1, U901.6 (Y)
- net TX-Z: now also J901.2, U901.7 (Z)
